File: schematic-big/TrackerFull/TrackerFull.kicad_pcb (KiCad board)
At the start: 2 copper layers, 41.1 x 38 mm, 57 parts, among them J1 Conn_01x05_Male, J3 Battery, J4 78646-3001, J5 USB power, Q2 DMG2305UXQ, Q3 DMG2305UXQ, SW1 PTS647SK38SMTR2LFS, U2 LIS3DSH, U3 ATtiny85-20PU, U4 MCP73831-2-OT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

Commit message: Last schematic changes
Parts:
- removed ANT1: 146235-0001, imported:ANT_1462350001
- removed H3, H4: MountingHole, MountingHole:MountingHole_2.2mm_M2
- removed J5: USB power, Connector_JST:JST_PH_B2B-PH-K_1x02_P2.00mm_Vertical
- added C20: 0.5 pF, Capacitor_SMD:C_0402_1005Metric, F.Cu at (187.7, 105.3)
- added C9: 1nF, Capacitor_SMD:C_0402_1005Metric, F.Cu at (186.2, 109.7)
- added E1: ANT-GNSSCP-TH18L1, imported:XDCR_ANT-GNSSCP-TH18L1, B.Cu at (186.7, 113.7)
- added J2: MUC-20PFFR-JS7001, imported:AMPHENOL_MUC-20PFFR-JS7001, B.Cu at (206.5, 73.4)
- added L4: 13nF, Inductor_SMD:L_0402_1005Metric, F.Cu at (187.2, 106.8)
- added L5: 6.2nH, Inductor_SMD:L_0402_1005Metric, F.Cu at (188.7, 107.9)
- C2: footprint Capacitor_SMD:C_0805_2012Metric -> Capacitor_SMD:C_0603_1608Metric
- FL1, L1, L3, R5, R6, U5: moved to F.Cu
- R9: footprint Resistor_SMD:R_0603_1608Metric -> Resistor_SMD:R_0402_1005Metric
- moved D3 30.6 mm to (200.8, 71.3), turned to 90 degrees
- moved R8 19.4 mm to (201.9, 73.4), turned to 270 degrees
- moved J4 17.7 mm to (175.7, 93.9), turned to 180 degrees
- moved L1 16.7 mm to (187.2, 103.6), turned to 270 degrees
- moved D2 16.4 mm to (201.8, 76.3)
- moved U5 15.3 mm to (187.4, 108.3), turned to 90 degrees
- moved SW1 15.0 mm to (179.0, 80.1), turned to 270 degrees
- moved L3 14.0 mm to (185.7, 103.9), turned to 180 degrees
- moved FL1 13.3 mm to (187.5, 109.9), turned to 270 degrees
- moved R6 12.2 mm to (185.7, 106.4), turned to 270 degrees
- moved Q3 12.1 mm to (186.2, 70.7), turned to 180 degrees
- moved C1 11.6 mm to (172.4, 86.4)
- moved U6 8.04 mm to (196.8, 92.1), turned to 0 degrees
- moved R5 7.52 mm to (178.6, 86.4), turned to 90 degrees
- moved C19 6.94 mm to (170.0, 85.0), turned to 90 degrees
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Connections:
- D1 pad 1: /AVR_SCK -> (no net)
- D1 pad 2: /AVR_MOSI_SDA -> (no net)
- D1 pad 23: /GPS_POWER -> /AVR_SCK
- D1 pad 24: (no net) -> /AVR_MOSI_SDA
- D1 pad 30: (no net) -> /GPS_POWER
- L1 pad 2: /GPS_SIGNAL -> Net-(C20-Pad1)
- L3 pad 1: /GPS_SIGNAL -> Net-(C20-Pad1)
- Q3 pad 2: BAT_IN -> /V_BAT
- Q3 pad 3: /V_BAT -> BAT_IN
- U5 pad 2: /GPS_POWER -> /2.5v
- U5 pad 6: /2.5v -> /GPS_POWER
Routing:
- net GNDREF: track 234.8 -> 142.6 mm, vias 34 -> 43
- net /AVR_SCK: track 26.0 -> 11.3 mm
- net /APW_OUT: track 39.1 -> 25.9 mm
- net /LED_CTL: track 7.71 -> 20.8 mm
- net /GPS_POWER: track 12.4 -> 1.72 mm
- net /AVR_MOSI_SDA: track 26.9 -> 19.1 mm
- net /SIM_IO: track 21.1 -> 14.2 mm
- net /GPS_RF: track 5.89 -> 0.01 mm, vias 1 -> 0
- net /ACCEL_CS: track 10.7 -> 4.93 mm, vias 1 -> 0
- net /AVR_RST: track 21.7 -> 26.7 mm
- net /SIM_RST: track 24.3 -> 19.6 mm
- net /HST_RXD: track 23.8 -> 19.2 mm
- net BAT_IN: track 72.5 -> 68.0 mm, vias 3 -> 5
- net /HST_TXD: track 28.5 -> 24.3 mm
- net Net-(D2-Pad2): track 5.58 -> 1.53 mm
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Other:
- board size 41.1 x 38 mm -> 41.1 x 61.5 mm
