File: schematic-big/TrackerFull/TrackerFull.sch (KiCad schematic (older format))
At the start: 61 parts, among them J1 Conn_01x05_Male, J3 Battery, J4 78646-3001, J5 USB power, Q2 DMG2305UXQ, Q3 DMG2305UXQ, SW1 PTS647SK38SMTR2LFS, U2 LIS3DSH, U3 ATtiny85-20PU, U4 MCP73831-2-OT, U5 BGU8019, U6 U.FL, U7 MIC5232-2.5YD5, U8 AP62301WU-7

Commit message: updated schematic
Parts:
- removed D7: D_Schottky, Diode_SMD:D_SMA, symbol Device:D_Schottky
- removed R2: 200K, Resistor_SMD:R_0603_1608Metric, symbol Device:R
- removed R4: 100K, Resistor_SMD:R_0805_2012Metric_Pad1.15x1.40mm_HandSolder, symbol Device:R
- C2: footprint Capacitor_SMD:C_0805_2012Metric -> Capacitor_SMD:C_0603_1608Metric
Connections:
- net labels removed: CHARGER_VDD
- wire segments 237 -> 235
- no-connect marks 26 -> 27
Other:
- moved on the sheet: C10, C11, C12, C13, C14, C15, C16, C17, C18, C6, C7, C8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

Commit message: Last schematic changes
Parts:
- removed ANT1: 146235-0001, ANT_1462350001, symbol 1462350001:1462350001
- removed H3, H4: MountingHole, MountingHole:MountingHole_2.2mm_M2, symbol Mechanical:MountingHole
- removed J5: USB power, Connector_JST:JST_PH_B2B-PH-K_1x02_P2.00mm_Vertical, symbol Connector:Screw_Terminal_01x02
- added C20: 0.5 pF, Capacitor_SMD:C_0402_1005Metric, symbol Device:C
- added E1: ANT-GNSSCP-TH18L1, XDCR_ANT-GNSSCP-TH18L1, symbol ANT-GNSSCP-TH18L1:ANT-GNSSCP-TH18L1
- added J2: MUC-20PFFR-JS7001, AMPHENOL_MUC-20PFFR-JS7001, symbol MUC-20PFFR-JS7001:MUC-20PFFR-JS7001
- added L4: 13nF, Inductor_SMD:L_0402_1005Metric, symbol Device:L
- added L5: 6.2nH, Inductor_SMD:L_0402_1005Metric, symbol Device:L
- added Q1: Q_NMOS_DGS, symbol Device:Q_NMOS_DGS
- C9: footprint (none) -> Capacitor_SMD:C_0402_1005Metric
- R9: footprint Resistor_SMD:R_0603_1608Metric -> Resistor_SMD:R_0402_1005Metric; Поле5 SR1-0603-220 -> CR0402-16W-2001FT
Connections:
- wire segments 235 -> 247
- no-connect marks 27 -> 31
Other:
- moved on the sheet: C9, J4, L1, L3, R6

Commit message: schematics update
Parts:
- removed C13: 100nF, Capacitor_SMD:C_0402_1005Metric, symbol Device:C
- removed C18: 22uF, Capacitor_SMD:C_0603_1608Metric, symbol Device:C
- removed Q1: Q_NMOS_DGS, symbol Device:Q_NMOS_DGS
- removed U8: AP62301WU-7, Package_TO_SOT_SMD:TSOT-23-6, symbol Regulator_Switching:AP62301
- added U1: TLV62585PDRLR, imported:SOT50P160X60-6N, symbol TLV62585PDRLR:TLV62585PDRLR
- C11, C2, C5: Поле5 C1608X6S1A106M080AC -> CL10A106KP8NQSC
- C17: footprint Capacitor_SMD:C_0603_1608Metric -> Capacitor_SMD:C_0805_2012Metric; Поле4 0.3 -> (none); Поле5 GRM188R61A226ME15D -> GRM21BD71A226ME44K
- L2: value MDWK4040T3R3MM -> 1uH; footprint Inductor_SMD:L_Taiyo-Yuden_MD-4040 -> Inductor_SMD:L_Vishay_IHLP-2020; Поле5 MDWK4040T3R3MM -> IHLP2020BZER1R0M01
- R1: footprint Resistor_SMD:R_0805_2012Metric_Pad1.15x1.40mm_HandSolder -> Resistor_SMD:R_0603_1608Metric; Поле5 RMCF0805JG100K -> CR161003F
- R13: value 43K -> 562K; Поле5 SR1-0603-343 -> CRCW0603562KFKEBC
- R14: value 10K -> 100K; footprint Resistor_SMD:R_0805_2012Metric_Pad1.15x1.40mm_HandSolder -> Resistor_SMD:R_0603_1608Metric; Поле5 CR0805-8W-103JT -> CR161003F
Connections:
- wire segments 247 -> 238
- no-connect marks 31 -> 34
Other:
- moved on the sheet: C17, J2

Commit message: replaced attiny
Parts:
- removed C4: 150nF, Capacitor_SMD:C_0402_1005Metric, symbol Device:C
- removed C5: 10uF, Capacitor_SMD:C_0603_1608Metric, symbol Device:C
- removed R11: 470, Resistor_SMD:R_0402_1005Metric, symbol Device:R
- removed U3: ATtiny85-20PU, Package_DIP:DIP-8_W7.62mm, symbol MCU_Microchip_ATtiny:ATtiny85-20SU
- added C13: 150nF, Capacitor_SMD:C_0402_1005Metric, symbol Device:C
- added C18: 10uF, Capacitor_SMD:C_0603_1608Metric, symbol Device:C
- added J5: Conn_01x04_Male, Connector_PinHeader_2.54mm:PinHeader_1x04_P2.54mm_Vertical, symbol Connector:Conn_01x04_Male
- added R2: 470, Resistor_SMD:R_0402_1005Metric, symbol Device:R
- added U8: ATtiny861A-MU, Package_DFN_QFN:QFN-32-1EP_5x5mm_P0.5mm_EP3.1x3.1mm, symbol MCU_Microchip_ATtiny:ATtiny861A-MU
- Q2, Q3: Поле5 DMG2305UXQ -> DMG2305UXQ-13
- U7: value MIC5232-2.5YD5 -> MIC5232-2.8YD5; Поле5 MIC5232-2.5YD5 -> MIC5232-2.8YD5
Connections:
- net ACCEL_INT1: now also U8.25 (PA1)
- net AVR_MOSI_SDA: now also U8.26 (PA0)
- net AVR_RST: now also J5.4 (Pin_4), U8.11 (~RESET~/PB7)
- net AVR_SCK: now also U8.23 (PA2)
- net BAT_IN: now also C13.2, C18.2, U8.18 (AVCC), U8.4 (VCC)
- net GNDREF: now also C13.1, C18.1, U8.21 (AGND), U8.33 (GND), U8.5 (GND)
- net LED_CTL: now also R3.2
- net PWR_CTRL: now also R2.1; no longer R3.1
- net V_BAT renamed BATTERY_IN
- new net: R3.1, U8.15 (PA5)
- new net: R2.2, U8.14 (PA6)
- new net ISP_MISO: J5.2 (Pin_2), U8.31 (PB1)
- new net ISP_MOSI: J5.3 (Pin_3), U8.30 (PB0)
- new net ISP_SCK: J5.1 (Pin_1), U8.32 (PB2)
- no-connect marks 34 -> 32
Other:
- moved on the sheet: J1, SW1

Commit message: replaced attiny
Connections:
- net AVR_MOSI_SDA: now also D1.2 (I2C2_SDA/IO20), U2.6 (SDA/SDI/SDO); no longer D1.24 (IO29)
- net AVR_SCK: now also D1.1 (I2C2_SCL/IO19), U2.4 (SCL/SPC); no longer D1.23 (LCD_SCK/IO16)
- net BATTERY_IN: now also Q3.3 (D); no longer Q3.2 (S)
- net BAT_IN: now also Q3.2 (S); no longer C15.1, C16.1, Q3.3 (D)
- net VBAT: now also C15.1, C16.1
- net ACCEL_CS: no longer names the net of R5.1, U2.8 (CS)
- net ACCEL_CS: now also U2.7 (SDO/SA0); no longer D1.19 (LCD_CS/IO15)
- net ACCEL_SCL: no longer names the net of D1.22 (LCD_SDO/IO18)
- net ACCEL_SCL: no longer U2.4 (SCL/SPC)
- net ACCEL_SDA: no longer names the net of D1.21 (LCD_DIO/IO17)
- net ACCEL_SDA: no longer U2.6 (SDA/SDI/SDO)
- net ACCEL_SDO: no longer names the net of D1.20 (LCD_RST/IO14)
- net ACCEL_SDO: no longer U2.7 (SDO/SA0)
- no-connect marks 32 -> 37
Other:
- moved on the sheet: C10, C12, C14, C15, C16, C8

Commit message: pcb layout
Parts:
- removed L1: LQG15HS5N1B02, Inductor_SMD:L_0402_1005Metric, symbol Device:L
- removed L3: LQG15HS1N8B02, Inductor_SMD:L_0402_1005Metric, symbol Device:L
- removed L5: 6.2nH, Inductor_SMD:L_0402_1005Metric, symbol Device:L
- added C4: 1.2 pF, Capacitor_SMD:C_0402_1005Metric, symbol Device:C
- added R11, R4: 0, Resistor_SMD:R_0402_1005Metric, symbol Device:R
- C20: value 0.5 pF -> 6.8 pF
- L4: value 13nF -> 6.2nH
- R10: value 10K -> 100K; footprint Resistor_SMD:R_0805_2012Metric_Pad1.15x1.40mm_HandSolder -> Resistor_SMD:R_0603_1608Metric; Поле5 CR0805-8W-103JT -> CR161003F
- U1: Поле5 (none) -> TLV62585PDRLR
Connections:
- net BAT_IN: now also R4.1; no longer C13.2, C18.2, C19.1, D5.3 (VDD), U7.1 (VIN), U7.3 (EN), U8.18 (AVCC), U8.4 (VCC)
- net GNDREF: now also R11.1; no longer C1.2, C13.1, C18.1, C19.2, C2.1, C20.2, C3.1, C9.2, D5.1 (VSS), E1.2, E1.3, E1.4, E1.5, FL1.2, FL1.3, FL1.5, J4.C5 (GND), J4.G1 (GND), J4.G2 (GND), J4.G3 (GND), J4.G4 (GND), J4.G5 (GND), J4.G6 (GND), R5.2, R6.1, SW1.3 (COM_1), SW1.4 (COM_2), U2.10 (GND), U2.12 (GND), U2.13 (ADC3), U2.16 (ADC1), U2.5 (GND), U5.1, U5.4, U7.2 (GND), U8.21 (AGND), U8.33 (GND), U8.5 (GND)
- net GPS_SIGNAL: now also L4.1, C4.1; no longer L4.2
- net at E1.1: now also C4.2
- net at C20.1: now also L4.2; no longer L4.1
- new net GNDD: C1.2, C13.1, C18.1, C19.2, C2.1, C20.2, C3.1, C9.2, D5.1 (VSS), E1.2, E1.3, E1.4, E1.5, FL1.2, FL1.3, FL1.5, J4.C5 (GND), J4.G1 (GND), J4.G2 (GND), J4.G3 (GND), J4.G4 (GND), J4.G5 (GND), J4.G6 (GND), R11.2, R5.2, R6.1, SW1.3 (COM_1), SW1.4 (COM_2), U2.10 (GND), U2.12 (GND), U2.13 (ADC3), U2.16 (ADC1), U2.5 (GND), U5.1, U5.4, U7.2 (GND), U8.21 (AGND), U8.33 (GND), U8.5 (GND)
- new net LOW_CURRENT: C13.2, C18.2, C19.1, D5.3 (VDD), R4.2, U7.1 (VIN), U7.3 (EN), U8.18 (AVCC), U8.4 (VCC)
Other:
- moved on the sheet: C20, E1, L4

Commit message: pcb layout
Parts:
- removed J4: 78646-3001, imported:MOLEX_78646-3001, symbol 78646-3001:78646-3001
- added J6: 78727-0001, simcard:Molex-78727-0001-0-0-MFG, symbol eec:78727-0001
- added Q1: DMG2305UXQ, Package_TO_SOT_SMD:SOT-23, symbol Transistor_FET:IRLML5203
- added R15: 100K, Resistor_SMD:R_0603_1608Metric, symbol Device:R
- E1: MANUFACTURER Linx -> (none); MAXIMUM_PACKAGE_HEIGHT 4 mm -> (none); PARTREV N/A -> (none); STANDARD Manufacturer Recommendations -> (none); Поле5 (none) -> ANT-GNSSCP-TH18L1
- FL1: Поле5 (none) -> SF14-1582M5UUD2
- SW1: Поле4 https://www.mouser.com/Search/Refine.aspx?Keyword=611-PTS64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 -> (none)
- U8: Поле5 (none) -> ATtiny861A-MU
Connections:
- net BAT_IN: now also R1.2, Q1.3 (D); no longer D3.1 (K), Q3.2 (S)
- net GNDD: now also J6.1 (GND3), J6.2 (GND2), J6.3 (GND1), J6.5 (GND4), J6.6 (GND5), J6.7 (DETECT_SPRING), J6.8 (GND6), J6.C5 (GND)
- net GNDREF: no longer R1.2
- net SIM_CLK: now also J6.C3 (CLK)
- net SIM_IO: now also J6.C7 (I/O)
- net SIM_RST: now also J6.C2 (RST)
- net VSIM: now also J6.C1 (VCC)
- new net POWER_INPUT: D3.1 (K), Q1.2 (S), Q3.2 (S), R15.1
- new net SIM_DETECT_LINE: J6.4 (DETECT_CONTACT), Q1.1 (G), R15.2
- no-connect marks 37 -> 38
Other:
- moved on the sheet: R4
Changed lines of the file:
@@
 Wire Wire Line
 	3000 6750 3000 6850
-Text GLabel 2950 7400 0    50   Input ~ 0
-BAT_IN
 Wire Wire Line
 	5200 1400 5200 1500
@@
 Wire Wire Line
 	3150 6650 3450 6650
-Wire Wire Line
-	2950 7300 2950 7400
 Text Label 1550 7100 0    50   ~ 0
 PWR_CTRL
@@
 Wire Wire Line
 	2400 7400 2400 7500
-$Comp
-L power:GNDREF #PWR01
-U 1 1 5F7617DA
-P 2400 7500
-F 0 "#PWR01" H 2400 7250 50  0001 C CNN
-F 1 "GNDREF" H 2405 7327 50  0000 C CNN
-F 2 "" H 2400 7500 50  0001 C CNN
-F 3 "" H 2400 7500 50  0001 C CNN
-	1    2400 7500
-	1    0    0    -1
-$EndComp
 Text Label 5500 3250 1    50   ~ 0
 CHARGER_PROG
-Text Label 3300 9550 0    50   ~ 0
-SIM_CLK
-Text Label 3300 9450 0    50   ~ 0
-SIM_RST
-Text Label 4700 9100 0    50   ~ 0
-VSIM
-Text Label 4700 9550 0    50   ~ 0
-SIM_IO
-Wire Wire Line
-	5250 9850 4650 9850
-NoConn ~ 4650 9250
-Wire Wire Line
-	4650 9150 4700 9150
-Wire Wire Line
-	4700 9150 4700 9100
-Wire Wire Line
-	4650 9550 4700 9550
-Wire Wire Line
-	3300 9550 3650 9550
-Wire Wire Line
-	3300 9450 3650 9450
 Wire Wire Line
 	3450 5750 3150 5750
@@
 Text Label 10400 3850 0    50   ~ 0
 VBAT
-Text GLabel 11150 2850 2    50   Input ~ 0
+Text GLabel 12000 2850 2    50   Input ~ 0
 BAT_IN
 NoConn ~ 4000 7500
@@
 Wire Wire Line
 	1900 3400 1900 3500
-Wire Wire Line
-	1900 3900 1900 4050
 Wire Wire Line
 	1900 3400 2150 3400
@@
 F 2 "PTS647SK38SMTR2LFS" H 8600 7350 50  0001 L BNN
 F 3 "https://www.digikey.com/en/products/detail/c-k/PTS-647-SK38-SMTR2-LFS/9649862" H 8600 7350 50  0001 L BNN
-F 4 "https://www.mouser.com/Search/Refine.aspx?Keyword=611-PTS647SK38SMTR2L" H 8600 7350 50  0001 L BNN "Поле4"
+F 4 "" H 8600 7350 50  0001 L BNN "Поле4"
 F 5 "611-PTS647SK38SMTR2L" H 8600 7350 50  0001 L BNN "Поле5"
 F 6 "3.8mm" H 8600 7350 50  0001 L BNN "Поле6"
@@
 	1    3200 6150
 	0    -1   -1   0
-$EndComp
-$Comp
-L 78646-3001:78646-3001 J4
-U 1 1 5F6BAE14
-P 4150 9450
-F 0 "J4" H 4150 10015 50  0000 C CNN
-F 1 "78646-3001" H 4150 9924 50  0000 C CNN
-F 2 "imported:MOLEX_78646-3001" H 4150 9450 50  0001 L BNN
-F 3 "https://www.digikey.in/product-detail/en/molex/0786463001/WM9364CT-ND/3770350?utm_source=snapeda&utm_medium=aggregator&utm_campaign=symbol" H 4150 9450 50  0001 L BNN
-F 4 "Conn Micro SIM Card SKT 6 POS 2.54mm Solder RA SMD 0.5A/Contact Embossed T/R" H 4150 9450 50  0001 L BNN "Поле4"
-F 5 "78646-3001" H 4150 9450 50  0001 L BNN "Поле5"
-F 6 "78646-3001" H 4150 9450 50  0001 L BNN "Поле6"
-F 7 "https://www.digikey.in/product-detail/en/molex/0786463001/WM9364CT-ND/3770350?utm_source=snapeda&utm_medium=aggregator&utm_campaign=symbol" H 4150 9450 50  0001 L BNN "Поле7"
-F 8 "None" H 4150 9450 50  0001 L BNN "Поле8"
-	1    4150 9450
-	1    0    0    -1
 $EndComp
 $Comp
@@
 Wire Wire Line
 	9900 2850 9900 2600
-Connection ~ 9900 2850
 Wire Wire Line
 	9900 2250 9900 2300
@@
 F 2 "Filter:Filter_1411-5_1.4x1.1mm" H 10550 9200 50  0001 C CNN
 F 3 "https://ru.mouser.com/datasheet/2/909/AVX_140127_Connectivity-1316412.pdf" H 10550 9200 50  0001 C CNN
+F 4 "SF14-1582M5UUD2" H 10550 9200 50  0001 C CNN "Поле5"
 	1    10550 9200
 	1    0    0    -1
@@
 F 2 "XDCR_ANT-GNSSCP-TH18L1" H 7050 8950 50  0001 L BNN
 F 3 "" H 7050 8950 50  0001 L BNN
-F 4 "Manufacturer Recommendations" H 7050 8950 50  0001 L BNN "STANDARD"
-F 5 "N/A" H 7050 8950 50  0001 L BNN "PARTREV"
-F 6 "4 mm" H 7050 8950 50  0001 L BNN "MAXIMUM_PACKAGE_HEIGHT"
-F 7 "Linx" H 7050 8950 50  0001 L BNN "MANUFACTURER"
+F 4 "" H 7050 8950 50  0001 L BNN "STANDARD"
+F 5 "" H 7050 8950 50  0001 L BNN "PARTREV"
+F 6 "" H 7050 8950 50  0001 L BNN "MAXIMUM_PACKAGE_HEIGHT"
+F 7 "" H 7050 8950 50  0001 L BNN "MANUFACTURER"
+F 8 "ANT-GNSSCP-TH18L1" H 7050 8950 50  0001 C CNN "Поле5"
 	1    7050 8950
 	1    0    0    -1
@@
 F 2 "Package_DFN_QFN:QFN-32-1EP_5x5mm_P0.5mm_EP3.1x3.1mm" H 7450 5950 50  0001 C CIN
 F 3 "http://ww1.microchip.com/downloads/en/DeviceDoc/doc8197.pdf" H 7450 5950 50  0001 C CNN
+F 4 "ATtiny861A-MU" H 7450 5950 50  0001 C CNN "Поле5"
 	1    7450 5950
 	1    0    0    -1
@@
 Connection ~ 10700 4450
 Connection ~ 11100 4450
-Wire Wire Line
-	9900 2850 10500 2850
 NoConn ~ 4200 7500
 Wire Wire Line
@@
 NoConn ~ 4600 7500
 NoConn ~ 4700 7500
-NoConn ~ 1150 6300
 $Comp
 L Device:C C4
@@
 L Device:R R4
 U 1 1 6004C267
-P 10500 3000
-F 0 "R4" H 10430 2954 50  0000 R CNN
-F 1 "0" H 10430 3045 50  0000 R CNN
-F 2 "Resistor_SMD:R_0402_1005Metric" H 10430 3091 50  0001 R CNN
-F 3 "https://www.digikey.com/en/products/detail/meritek/CR20000J/13410265" H 10500 3000 50  0001 C CNN
-F 4 "CR20000J" H 10500 3000 50  0001 C CNN "Поле5"
-	1    10500 3000
-	1    0    0    -1
-$EndComp
-Connection ~ 10500 2850
-Wire Wire Line
-	10500 2850 11150 2850
-Wire Wire Line
-	10500 3150 10500 3350
-Text Label 10500 3350 0    50   ~ 0
+P 11350 3000
+F 0 "R4" H 11280 2954 50  0000 R CNN
+F 1 "0" H 11280 3045 50  0000 R CNN
+F 2 "Resistor_SMD:R_0402_1005Metric" H 11280 3091 50  0001 R CNN
+F 3 "https://www.digikey.com/en/products/detail/meritek/CR20000J/13410265" H 11350 3000 50  0001 C CNN
+F 4 "CR20000J" H 11350 3000 50  0001 C CNN "Поле5"
+	1    11350 3000
+	1    0    0    -1
+$EndComp
+Connection ~ 11350 2850
+Wire Wire Line
+	11350 2850 12000 2850
+Wire Wire Line
+	11350 3150 11350 3350
+Text Label 11350 3350 0    50   ~ 0
 LOW_CURRENT
 Text Label 650  1250 0    50   ~ 0
@@
 $EndComp
 $Comp
-L power:GNDD #PWR0115
-U 1 1 60150F85
-P 5250 9850
-F 0 "#PWR0115" H 5250 9600 50  0001 C CNN
-F 1 "GNDD" H 5254 9695 50  0000 C CNN
-F 2 "" H 5250 9850 50  0001 C CNN
-F 3 "" H 5250 9850 50  0001 C CNN
-	1    5250 9850
-	1    0    0    -1
-$EndComp
-$Comp
 L power:GNDD #PWR0116
 U 1 1 60162517
@@
 	1    0    0    -1
 $EndComp
+Wire Wire Line
+	2950 7300 2950 7500
+Wire Wire Line
+	2400 7500 2950 7500
+Connection ~ 2950 7500
+Wire Wire Line
+	2950 7500 2950 7750
+Text Label 14650 4950 0    50   ~ 0
+VSIM
+Text GLabel 2950 7650 0    50   Input ~ 0
+BAT_IN
+Wire Wire Line
+	1900 3900 1900 4050
+Text Label 10350 3400 0    50   ~ 0
+SIM_DETECT_LINE
+$Comp
+L Transistor_FET:IRLML5203 Q1
+U 1 1 5FB77A47
+P 10350 2950
+F 0 "Q1" H 10554 2996 50  0000 L CNN
+F 1 "DMG2305UXQ" H 10554 2905 50  0000 L CNN
+F 2 "Package_TO_SOT_SMD:SOT-23" H 10550 2875 50  0001 L CIN
+F 3 "https://www.diodes.com/assets/Datasheets/DMG2305UXQ.pdf" H 10350 2950 50  0001 L CNN
+F 4 "DMG2305UXQ-13 " H 10350 2950 50  0001 C CNN "Поле5"
+	1    10350 2950
+	0    1    -1   0
+$EndComp
+Wire Wire Line
+	9900 2850 10000 2850
+Connection ~ 9900 2850
+Wire Wire Line
+	10550 2850 11350 2850
+$Comp
+L Device:R R15
+U 1 1 5FB9E73A
+P 10000 3100
+F 0 "R15" H 9950 3100 50  0000 L CNN
+F 1 "100K" H 9850 3000 50  0000 L CNN
+F 2 "Resistor_SMD:R_0603_1608Metric" H 10070 3009 50  0001 L CNN
+F 3 "https://www.digikey.com/en/products/detail/meritek/CR161003F/13412806" H 10000 3100 50  0001 C CNN
+F 4 "CR161003F" H 10000 3100 50  0001 C CNN "Поле5"
+	1    10000 3100
+	1    0    0    -1
+$EndComp
+Wire Wire Line
+	10000 2850 10000 2950
+Connection ~ 10000 2850
+Wire Wire Line
+	10000 2850 10150 2850
+Wire Wire Line
+	10000 3250 10350 3250
+Wire Wire Line
+	10350 3250 10350 3150
+Wire Wire Line
+	10350 3400 10350 3250
+Connection ~ 10350 3250
+$Comp
+L power:GNDD #PWR0115
+U 1 1 5FB652B8
+P 2500 9050
+F 0 "#PWR0115" H 2500 8800 50  0001 C CNN
+F 1 "GNDD" H 2504 8895 50  0000 C CNN
+F 2 "" H 2500 9050 50  0001 C CNN
+F 3 "" H 2500 9050 50  0001 C CNN
+	1    2500 9050
+	1    0    0    -1
+$EndComp
+Wire Wire Line
+	1850 9050 2500 9050
+Text Label 2300 8450 0    50   ~ 0
+SIM_DETECT_LINE
+Wire Wire Line
+	1850 8450 2500 8450
+$Comp
+L power:GNDD #PWR0128
+U 1 1 5FDBC25C
+P 2000 8050
+F 0 "#PWR0128" H 2000 7800 50  0001 C CNN
+F 1 "GNDD" H 2004 7895 50  0000 C CNN
+F 2 "" H 2000 8050 50  0001 C CNN
+F 3 "" H 2000 8050 50  0001 C CNN
+	1    2000 8050
+	1    0    0    -1
+$EndComp
+$Comp
+L power:GNDD #PWR0127
+U 1 1 5FDBBE37
+P 2000 8750
+F 0 "#PWR0127" H 2000 8500 50  0001 C CNN
+F 1 "GNDD" H 2004 8595 50  0000 C CNN
+F 2 "" H 2000 8750 50  0001 C CNN
+F 3 "" H 2000 8750 50  0001 C CNN
+	1    2000 8750
+	1    0    0    -1
+$EndComp
+$Comp
+L power:GNDD #PWR0126
+U 1 1 5FDBB7BC
+P 2000 9250
+F 0 "#PWR0126" H 2000 9000 50  0001 C CNN
+F 1 "GNDD" H 2100 9250 50  0000 C CNN
+F 2 "" H 2000 9250 50  0001 C CNN
+F 3 "" H 2000 9250 50  0001 C CNN
+	1    2000 9250
+	1    0    0    -1
+$EndComp
+Wire Wire Line
+	1850 8050 2000 8050
+Wire Wire Line
+	1850 8750 1850 8850
+Connection ~ 1850 8750
+Wire Wire Line
+	1850 8750 2000 8750
+Wire Wire Line
+	1850 9250 2000 9250
+Wire Wire Line
+	1850 9450 2000 9450
+Wire Wire Line
+	1850 9650 2000 9650
+Wire Wire Line
+	1850 9850 2000 9850
+Wire Wire Line
+	1850 10650 2000 10650
+NoConn ~ 1850 10850
+Text Label 2000 10650 0    50   ~ 0
+SIM_IO
+NoConn ~ 1850 10450
+$Comp
+L power:GNDD #PWR0125
+U 1 1 5FD18DCB
+P 2150 10250
+F 0 "#PWR0125" H 2150 10000 50  0001 C CNN
+F 1 "GNDD" H 2154 10095 50  0000 C CNN
+F 2 "" H 2150 10250 50  0001 C CNN
+F 3 "" H 2150 10250 50  0001 C CNN
+	1    2150 10250
+	1    0    0    -1
+$EndComp
+Wire Wire Line
+	1850 10250 2150 10250
+NoConn ~ 1850 10050
+Text Label 2000 9850 0    50   ~ 0
+SIM_CLK
+Text Label 2000 9650 0    50   ~ 0
+SIM_RST
+Text Label 2000 9450 0    50   ~ 0
+VSIM
+Wire Wire Line
+	1850 8650 1850 8750
+Connection ~ 1850 8050
+Wire Wire Line
+	1850 8250 1850 8050
+Wire Wire Line
+	1850 7850 1850 8050
+$Comp
+L eec:78727-0001 J6
+U 1 1 5FC4195D
+P 1950 7850
+F 0 "J6" H 1258 8215 50  0000 C CNN
+F 1 "78727-0001" H 1258 8124 50  0000 C CNN
+F 2 "simcard:Molex-78727-0001-0-0-MFG" H 1950 8350 50  0001 L CNN
+F 3 "https://www.molex.com/webdocs/datasheets/pdf/en-us/0787270001_MEMORY_CARD_SOCKET.pdf" H 1950 8450 50  0001 L CNN
+F 4 "78727-0001" H 1950 7850 50  0001 C CNN "Поле5"
+	1    1950 7850
+	1    0    0    -1
+$EndComp
+Text Label 9800 2850 0    50   ~ 0
+POWER_INPUT
 $EndSCHEMATC

Commit message: rf
Parts:
- C20: Поле5 (none) -> GRM1555C1E6R8CA01D
- C4: Поле5 (none) -> GRM1555C1H1R2BA01D
- C9: Поле5 (none) -> GRM1555C2A102JE01D
- L4: Поле5 (none) -> LQW15AN6N2B0ZD
Connections:
- net LNA_OUTPUT: now reaches FL1.1, U5.3
- net ANT_OUT: now reaches C4.2, E1.1
Other:
- moved on the sheet: C10, C12, C14, C15, C16, C8
