File: schematic-big/TrackerFull/TrackerFull.sch (KiCad schematic (older format))
At the start: 66 parts, among them J1 Conn_01x05_Male, J2 USB, J3 Battery, J5 Conn_01x04_Male, J6 78727-0001, Q1 DMG2305UXQ, Q2 DMG2305UXQ, Q3 DMG2305UXQ, Q4 DMN60H080DS, U1 TLV62585PDRLR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

Commit message: last pcb version
Connections:
- net CHARGER_STAT: now also U8.25 (PA1); no longer D1.19 (LCD_CS/IO15)
- net at D1.20 (LCD_RST/IO14): no longer R17.2
- net at U8.2 (PB3): now also R17.2
Other:
- moved on the sheet: R17
Changed lines of the file:
@@
 NoConn ~ 4100 7500
 Wire Wire Line
-	4300 7900 4300 8100
-Text Label 4300 8100 3    50   ~ 0
+	8550 6350 8750 6350
+Text Label 8750 6350 0    50   ~ 0
 +5V
 NoConn ~ 3450 5950
@@
 NoConn ~ 3450 6350
 Wire Wire Line
-	4200 7500 4200 8000
-Text Label 4200 8000 3    50   ~ 0
+	8150 5250 8650 5250
+Text Label 8650 5250 0    50   ~ 0
 CHARGER_STAT
 $Comp
@@
 Connection ~ 2400 7100
 Wire Wire Line
-	4300 7600 4300 7500
+	8250 6350 8150 6350
 Text Label 5800 6850 2    50   ~ 0
 GPS_POWER
@@
 Text Label 7100 8700 0    50   ~ 0
 ANT_OUT
-NoConn ~ 8150 6350
 NoConn ~ 8150 5850
 NoConn ~ 8150 5550
@@
 L Device:R R17
 U 1 1 5F85A184
-P 4300 7750
-F 0 "R17" V 4400 7800 50  0000 R CNN
-F 1 "10K" V 4300 7800 50  0000 R CNN
-F 2 "Resistor_SMD:R_0603_1608Metric" H 4230 7841 50  0001 R CNN
-F 3 "https://www.digikey.com/en/products/detail/stackpole-electronics-inc/RMCF0603FG10K0/1761236" H 4300 7750 50  0001 C CNN
-F 4 "RMCF0603FG10K0" H 4300 7750 50  0001 C CNN "Поле5"
-	1    4300 7750
-	-1   0    0    1
+P 8400 6350
+F 0 "R17" V 8500 6400 50  0000 R CNN
+F 1 "10K" V 8400 6400 50  0000 R CNN
+F 2 "Resistor_SMD:R_0603_1608Metric" H 8330 6441 50  0001 R CNN
+F 3 "https://www.digikey.com/en/products/detail/stackpole-electronics-inc/RMCF0603FG10K0/1761236" H 8400 6350 50  0001 C CNN
+F 4 "RMCF0603FG10K0" H 8400 6350 50  0001 C CNN "Поле5"
+	1    8400 6350
+	0    1    1    0
 $EndComp
 $Comp
@@
 	1    0    0    -1
 $EndComp
-NoConn ~ 8150 5250
 Wire Wire Line
 	9900 2850 10150 2850
@@
 Text Label 7450 3950 0    50   ~ 0
 2.5v
-NoConn ~ 8150 5450
 Text Label 9400 6750 0    50   ~ 0
 2.5v
@@
 NoConn ~ 3450 6150
 NoConn ~ 3450 6450
+NoConn ~ 8150 5450
+NoConn ~ 4200 7500
+NoConn ~ 4300 7500
 $EndSCHEMATC

Commit message: fixes
Parts:
- added R21: 10K, Resistor_SMD:R_0402_1005Metric, symbol Device:R
Connections:
- net GNDD: now also R21.2
- net at R17.2, U8.2 (PB3): now also R21.1
Other:
- moved on the sheet: R17
Changed lines of the file:
@@
 NoConn ~ 4100 7500
 Wire Wire Line
-	8550 6350 8750 6350
-Text Label 8750 6350 0    50   ~ 0
+	9800 5800 9800 5600
+Text Label 9800 5750 0    50   ~ 0
 +5V
 NoConn ~ 3450 5950
@@
 Connection ~ 2400 7100
 Wire Wire Line
-	8250 6350 8150 6350
+	9800 6100 9800 6150
 Text Label 5800 6850 2    50   ~ 0
 GPS_POWER
@@
 L Device:R R17
 U 1 1 5F85A184
-P 8400 6350
-F 0 "R17" V 8500 6400 50  0000 R CNN
-F 1 "10K" V 8400 6400 50  0000 R CNN
-F 2 "Resistor_SMD:R_0603_1608Metric" H 8330 6441 50  0001 R CNN
-F 3 "https://www.digikey.com/en/products/detail/stackpole-electronics-inc/RMCF0603FG10K0/1761236" H 8400 6350 50  0001 C CNN
-F 4 "RMCF0603FG10K0" H 8400 6350 50  0001 C CNN "Поле5"
-	1    8400 6350
-	0    1    1    0
+P 9800 5950
+F 0 "R17" V 9900 6000 50  0000 R CNN
+F 1 "10K" V 9800 6000 50  0000 R CNN
+F 2 "Resistor_SMD:R_0603_1608Metric" H 9730 6041 50  0001 R CNN
+F 3 "https://www.digikey.com/en/products/detail/stackpole-electronics-inc/RMCF0603FG10K0/1761236" H 9800 5950 50  0001 C CNN
+F 4 "RMCF0603FG10K0" H 9800 5950 50  0001 C CNN "Поле5"
+	1    9800 5950
+	1    0    0    -1
 $EndComp
 $Comp
@@
 NoConn ~ 4200 7500
 NoConn ~ 4300 7500
+$Comp
+L Device:R R21
+U 1 1 6016E277
+P 9800 6350
+F 0 "R21" V 9900 6400 50  0000 R CNN
+F 1 "10K" V 9800 6400 50  0000 R CNN
+F 2 "Resistor_SMD:R_0402_1005Metric" H 9730 6441 50  0001 R CNN
+F 3 "" H 9800 6350 50  0001 C CNN
+F 4 "" H 9800 6350 50  0001 C CNN "Поле5"
+	1    9800 6350
+	1    0    0    -1
+$EndComp
+Wire Wire Line
+	8150 6350 9000 6350
+Wire Wire Line
+	9000 6350 9000 6150
+Wire Wire Line
+	9000 6150 9800 6150
+Connection ~ 9800 6150
+Wire Wire Line
+	9800 6150 9800 6200
+$Comp
+L power:GNDD #PWR0124
+U 1 1 60184AAA
+P 9800 6600
+F 0 "#PWR0124" H 9800 6350 50  0001 C CNN
+F 1 "GNDD" H 9804 6445 50  0000 C CNN
+F 2 "" H 9800 6600 50  0001 C CNN
+F 3 "" H 9800 6600 50  0001 C CNN
+	1    9800 6600
+	1    0    0    -1
+$EndComp
+Wire Wire Line
+	9800 6500 9800 6600
 $EndSCHEMATC
